Commit message: i hate blax and also here is urdf and config ig

File: src/sim_folder/src/robohub/description/urdf/robot.urdf.xacro (robot description, xacro)
@@ -2,3 +2,4 @@
 <robot xmlns:xacro="http://www.ros.org/wiki/xacro" name="my_robot">
   <xacro:include filename="robot_core.xacro"/>
+  <xacro:include filename="../gazebo_control.xacro"/>
 </robot>

File: src/sim_folder/src/robohub/description/urdf/robot_core.xacro (robot description, xacro)
@@ -85,4 +85,7 @@
         </xacro:inertial_box>
     </link>
+    <gazebo reference="kropp">
+        <material>Gazebo/White</material>
+    </gazebo>
     <!-- Gimbal ("gimble")
          Ønsket: blå stand er fast, og orange boks roterer (yaw rundt Z, pitch rundt X). -->
@@ -109,4 +112,7 @@
         </xacro:inertial_cylinder>
     </link>
+    <gazebo reference="gimble_stand">
+        <material>Gazebo/Blue</material>
+    </gazebo>
     <joint name="gimble_yaw_joint" type="continuous">
         <parent link="gimble_stand"/>
@@ -150,4 +156,7 @@
         </xacro:inertial_box>
     </link>
+    <gazebo reference="lidar">
+        <material>Gazebo/Orange</material>
+    </gazebo>
     <!-- ===================== -->
     <!-- 3) Wheels (drivhjul + støttehjul/caster) -->
@@ -181,4 +190,7 @@
         </xacro:inertial_cylinder>
     </link>
+    <gazebo reference="venstre_hjul">
+        <material>Gazebo/Black</material>
+    </gazebo>
     <joint name="høyre_hjul_joint" type="continuous">
         <parent link="kropp"/>
@@ -206,4 +218,7 @@
         </xacro:inertial_cylinder>
     </link>
+    <gazebo reference="høyre_hjul">
+        <material>Gazebo/Black</material>
+    </gazebo>
     <!-- Støttehjul (caster)
          For en enkel plattform brukes et fast montert "kulehjul" (sphere) for stabil støtte.
@@ -230,3 +245,9 @@
         </xacro:inertial_sphere>
     </link>
+    <gazebo reference="cast_hjul">
+        <material>Gazebo/Black</material>
+        <!--friksjons coff-->
+        <mu1 value="0.000001"/>
+        <mu2 value="0.000001"/>
+    </gazebo>
 </robot>
