Commit message: Ros translation funke no, data overføres. Husk at for å kjør lidar, så må kommandoen 'gz model -m two_wheel_robot -l lidar_link' kjøres etter du har starta sim for å funk.

File: src/sim_folder/src/simulation_package/gazebo_includes/models/full_robot.urdf (robot description, URDF)
Before this commit: robot my_robot, 9 links, 8 joints
Joints:
- joint base_to_offset: child footbase_link -> base_link; origin xyz=0.0 0.85 0.2 rpy=0 0 0 -> xyz=0.0 0.0 0.85 rpy=0 0 0; parent base_link -> footbase_link

File: src/sim_folder/src/simulation_package/gazebo_urdf/robot.urdf.xacro (robot description, xacro)
@@ -7,4 +7,14 @@
   <!--> Components </!-->
   <xacro:include filename="component_bases/lidar_base.xacro"/>
+  <plugin
+    filename="gz-sim-diff-drive-system"
+    name="gz::sim::systems::DiffDrive">
+    <left_joint>venstre_hjul_joint</left_joint>
+    <right_joint>høyre_hjul_joint</right_joint>
+    <wheel_separation>0.205</wheel_separation>
+    <wheel_radius>0.035</wheel_radius>
+    <odom_publish_frequency>1</odom_publish_frequency>
+    <topic>cmd_vel</topic>
+  </plugin>
   <!--> Control units </!-->
   <!-->

File: src/sim_folder/src/simulation_package/gazebo_urdf/vehicle_bases/chassis_base.xacro (robot description, xacro)
@@ -7,5 +7,5 @@
         <parent link="footbase_link"/>
         <child link="base_link"/>
-        <origin xyz="0.0 0.0 0.85" rpy="0 0 0"/>  <!-- This is the offset: 10cm forward, 20cm up -->
+        <origin xyz="0.0 0.0 0.085" rpy="0 0 0"/>  <!-- This is the offset: 10cm forward, 20cm up -->
     </joint>
     <joint name="kropp_joint" type="fixed">
