Commit message: Fikk robot_state_publisher til å funk, woop woop. Vises i rviz2

File: src/wg_navigation/params/URDF/URDF_ASSEMBLY.urdf (robot description, URDF)
Before this commit: robot URDF_ASSEMBLY, 20 links, 19 joints
Links:
- removed link base_link-v5
- added link base_footprint
- added link base_link
- added link chassis_link, mass 2.60032387092806; collision mesh filename=package://wg_navigation/URDF/base_link-v5.stl scale=0.001 0.001 0.001; visual mesh filename=package://wg_navigation/URDF/base_link-v5.stl scale=0.001 0.001 0.001
- link Cam-V2.1-v1-v1: geometry collision mesh filename=package://wg_navigation/URDF/Cam-V2.1-v1-v1.stl scale=0.001 0.001 0.001; visual mesh filename=package://wg_navigation/URDF/Cam-V2.1-v1-v1.stl scale=0.001 0.001 0.001
- link LD06_LiDAR-v9: geometry collision mesh filename=package://wg_navigation/URDF/LD06_LiDAR-v9.stl scale=0.001 0.001 0.001; visual mesh filename=package://wg_navigation/URDF/LD06_LiDAR-v9.stl scale=0.001 0.001 0.001
- link Sharp_IR-Sensor-v1: geometry collision mesh filename=package://wg_navigation/URDF/Sharp_IR-Sensor-v1.stl scale=0.001 0.001 0.001; visual mesh filename=package://wg_navigation/URDF/Sharp_IR-Sensor-v1.stl scale=0.001 0.001 0.001
- link beltestrammer-wide-BB-left-v6: geometry collision mesh filename=package://wg_navigation/URDF/beltestrammer-wide-BB-left-v6.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 scale=0.001 0.001 0.001; visual mesh filename=package://wg_navigation/URDF/beltestrammer-wide-BB-left-v6.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 scale=0.001 0.001 0.001
- link beltestrammer-wide-BB-right-v2: geometry collision mesh filename=package://wg_navigation/URDF/beltestrammer-wide-BB-right-v2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 scale=0.001 0.001 0.001; visual mesh filename=package://wg_navigation/URDF/beltestrammer-wide-BB-right-v2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 scale=0.001 0.001 0.001
- link distance-sensor-holder-v3: geometry collision mesh filename=package://wg_navigation/URDF/distance-sensor-holder-v3.stl scale=0.001 0.001 0.001; visual mesh filename=package://wg_navigation/URDF/distance-sensor-holder-v3.stl scale=0.001 0.001 0.001
- link drivewheel-right: geometry collision mesh filename=package://wg_navigation/URDF/drivewheel-right.stl scale=0.001 0.001 0.001; visual mesh filename=package://wg_navigation/URDF/drivewheel-right.stl scale=0.001 0.001 0.001
- link drivewheel_left: geometry collision mesh filename=package://wg_navigation/URDF/drivewheel_left.stl scale=0.001 0.001 0.001; visual mesh filename=package://wg_navigation/URDF/drivewheel_left.stl scale=0.001 0.001 0.001
- link left_back_axle: geometry collision mesh filename=package://wg_navigation/URDF/left_back_axle.stl scale=0.001 0.001 0.001; visual mesh filename=package://wg_navigation/URDF/left_back_axle.stl scale=0.001 0.001 0.001
- link left_back_rullehjul: geometry collision mesh filename=package://wg_navigation/URDF/left_back_rullehjul.stl scale=0.001 0.001 0.001; visual mesh filename=package://wg_navigation/URDF/left_back_rullehjul.stl scale=0.001 0.001 0.001
- link left_front_axle: geometry collision mesh filename=package://wg_navigation/URDF/left_front_axle.stl scale=0.001 0.001 0.001; visual mesh filename=package://wg_navigation/URDF/left_front_axle.stl scale=0.001 0.001 0.001
- link left_right_rullehjul: geometry collision mesh filename=package://wg_navigation/URDF/left_right_rullehjul.stl scale=0.001 0.001 0.001; visual mesh filename=package://wg_navigation/URDF/left_right_rullehjul.stl scale=0.001 0.001 0.001
- link lidar-tilt-mount-v1: geometry collision mesh filename=package://wg_navigation/URDF/lidar-tilt-mount-v1.stl scale=0.001 0.001 0.001; visual mesh filename=package://wg_navigation/URDF/lidar-tilt-mount-v1.stl scale=0.001 0.001 0.001
- link lidar-tilt-v2: geometry collision mesh filename=package://wg_navigation/URDF/lidar-tilt-v2.stl scale=0.001 0.001 0.001; visual mesh filename=package://wg_navigation/URDF/lidar-tilt-v2.stl scale=0.001 0.001 0.001
- link right_back_axle: geometry collision mesh filename=package://wg_navigation/URDF/right_back_axle.stl scale=0.001 0.001 0.001; visual mesh filename=package://wg_navigation/URDF/right_back_axle.stl scale=0.001 0.001 0.001
- link right_back_rullehjul: geometry collision mesh filename=package://wg_navigation/URDF/right_back_rullehjul.stl scale=0.001 0.001 0.001; visual mesh filename=package://wg_navigation/URDF/right_back_rullehjul.stl scale=0.001 0.001 0.001
- link right_front_axle: geometry collision mesh filename=package://wg_navigation/URDF/right_front_axle.stl scale=0.001 0.001 0.001; visual mesh filename=package://wg_navigation/URDF/right_front_axle.stl scale=0.001 0.001 0.001
- link right_front_rullehjul: geometry collision mesh filename=package://wg_navigation/URDF/right_front_rullehjul.stl scale=0.001 0.001 0.001; visual mesh filename=package://wg_navigation/URDF/right_front_rullehjul.stl scale=0.001 0.001 0.001
- link standoff-cam-v1: geometry collision mesh filename=package://wg_navigation/URDF/standoff-cam-v1.stl scale=0.001 0.001 0.001; visual mesh filename=package://wg_navigation/URDF/standoff-cam-v1.stl scale=0.001 0.001 0.001
Joints:
- added joint base_footprint_link: type fixed, parent base_link, child base_footprint, origin xyz=0 0 -0.405
- added joint rigid_base_link: type fixed, parent base_link, child chassis_link, origin xyz=0 0 0 rpy=0 0 0
- joint base_link-v5_Rigid-1: parent base_link-v5 -> chassis_link
- joint base_link-v5_Rigid-2: parent base_link-v5 -> chassis_link
- joint base_link-v5_Rigid-21: parent base_link-v5 -> chassis_link
- joint base_link-v5_Rigid-31: parent base_link-v5 -> chassis_link
- joint base_link-v5_Rigid-33: parent base_link-v5 -> chassis_link
- joint base_link-v5_Rigid-34: parent base_link-v5 -> chassis_link
- joint base_link-v5_Rigid-35: parent base_link-v5 -> chassis_link
- joint base_link-v5_Rigid-36: parent base_link-v5 -> chassis_link

Commit message: Fiksa et par problema i startup sjiten.

File: src/wg_navigation/params/URDF/URDF_ASSEMBLY.urdf (robot description, URDF)
Before this commit: robot URDF_ASSEMBLY, 22 links, 21 joints
Joints:
- joint base_footprint_link: origin xyz=0 0 -0.405 -> xyz=0 0 -0.05

Commit message: Fiksa URDF

File: src/wg_navigation/params/URDF/URDF_ASSEMBLY.urdf (robot description, URDF)
Before this commit: robot URDF_ASSEMBLY, 23 links, 23 joints
Joints:
- removed joint beltestrammer-wide-BB-left-v6_Revolute-4
- removed joint beltestrammer-wide-BB-right-v2_Revolute-3
- added joint left_wheel_joint: type continuous, parent beltestrammer-wide-BB-left-v6, child drivewheel_left, origin xyz=0.0 2.220446049250313e-18 0.006300000000000008 rpy=3.141592653589793 -0.0 0.0, axis -6.162975822039155e-33 2.1005126272699612e-48 0.9999999999999999
- added joint right_wheel_joint: type continuous, parent beltestrammer-wide-BB-right-v2, child drivewheel-right, origin xyz=0.0 2.220446049250313e-18 -0.0062999999999999905 rpy=3.141592653589793 -0.0 0.0, axis -6.162975822039155e-33 2.1005126272699612e-48 0.9999999999999999

Commit message: Faaaaaaaaaaaaaaaaaaaaaaaaaaakk oooooooooooooooooooff. kanskje no.

File: src/wg_navigation/params/URDF/URDF_ASSEMBLY.urdf (robot description, URDF)
Before this commit: robot URDF_ASSEMBLY, 23 links, 23 joints
Links:
- removed link drivewheel-right
- added link drivewheel_right, mass 0.2722552771680154; collision mesh filename=package://wg_navigation/URDF/drivewheel-right.stl scale=0.001 0.001 0.001; visual mesh filename=package://wg_navigation/URDF/drivewheel-right.stl scale=0.001 0.001 0.001
Joints:
- joint right_wheel_joint: child drivewheel-right -> drivewheel_right

Commit message: Fiksa dobbel link urdf kanskje.

File: src/wg_navigation/params/URDF/URDF_ASSEMBLY.urdf (robot description, URDF)
Before this commit: robot URDF_ASSEMBLY, 23 links, 23 joints
Joints:
- removed joint base_laser_to_lidar
- removed joint base_link_to_base_laser

Commit message: bruh

File: src/wg_navigation/params/URDF/URDF_ASSEMBLY.urdf (robot description, URDF)
Before this commit: robot URDF_ASSEMBLY, 22 links, 21 joints
Links:
- removed link base_laser
- added link base_link
